Commit message: fix livox name
Signed-off-by: Yukihiro Saito <yukky.saito@gmail.com>

File: livox_description/urdf/livox_horizon.xacro (robot description, xacro)
@@ -4,10 +4,10 @@
     <xacro:property name="sensor_box" value="0.1" />
     <xacro:property name="mass" value="0.01" />
-    <joint name="${suffix}_joint" type="fixed">
+    <joint name="${suffix}_base_mount_joint" type="fixed">
       <origin rpy="${roll} ${pitch} ${yaw}" xyz="${x} ${y} ${z}"/>
       <parent link="${parent}"/>
-      <child  link="${suffix}_link"/>
+      <child  link="${suffix}_base_link"/>
     </joint>
-    <link name="${suffix}_link">
+    <link name="${suffix}_base_link">
       <visual>
         <geometry>
@@ -33,4 +33,16 @@
       </collision> -->
     </link>
+    <joint name="${suffix}_base_scan_joint" type="fixed" >
+      <origin xyz="0 0 0.0377" rpy="0 0 0" />
+      <parent link="${suffix}_base_link" />
+      <child link="${suffix}"/>
+    </joint>
+    <link name="${suffix}">
+      <inertial>
+        <mass value="0.0"/>
+        <origin xyz="0 0 0"/>
+        <inertia ixx="0" ixy="0" ixz="0" iyy="0" iyz="0" izz="0"/>
+      </inertial>
+    </link>
   </xacro:macro>
 </robot>
