Commit message: change to velodyne_front -> velodyne_top

File: aip_x1_description/urdf/sensor_kit.xacro (robot description, xacro)
@@ -17,6 +17,6 @@
     <xacro:property name="calibration" value="${load_yaml('$(arg config_dir)/sensor_kit_calibration.yaml')}"/>
     <!-- lidar -->
-    <VLP-16 parent="sensor_kit_base_link" name="velodyne_front" topic="/points_raw" hz="10" samples="220" gpu="$(arg gpu)">
-      <origin xyz="${calibration['sensor_kit_base_link2velodyne_front_base_link']['x']} ${calibration['sensor_kit_base_link2velodyne_front_base_link']['y']} ${calibration['sensor_kit_base_link2velodyne_front_base_link']['z']}" rpy="${calibration['sensor_kit_base_link2velodyne_front_base_link']['roll']} ${calibration['sensor_kit_base_link2velodyne_front_base_link']['pitch']} ${calibration['sensor_kit_base_link2velodyne_front_base_link']['yaw']}" />
+    <VLP-16 parent="sensor_kit_base_link" name="velodyne_top" topic="/points_raw" hz="10" samples="220" gpu="$(arg gpu)">
+      <origin xyz="${calibration['sensor_kit_base_link2velodyne_top_base_link']['x']} ${calibration['sensor_kit_base_link2velodyne_top_base_link']['y']} ${calibration['sensor_kit_base_link2velodyne_top_base_link']['z']}" rpy="${calibration['sensor_kit_base_link2velodyne_top_base_link']['roll']} ${calibration['sensor_kit_base_link2velodyne_top_base_link']['pitch']} ${calibration['sensor_kit_base_link2velodyne_top_base_link']['yaw']}" />
     </VLP-16>
     <xacro:include filename="$(find livox_description)/urdf/livox_horizon.xacro"/>

Commit message: refactor code

File: aip_x1_description/urdf/sensor_kit.xacro (robot description, xacro)
@@ -3,5 +3,4 @@
   <xacro:macro name="sensor_kit_macro" params="parent x y z roll pitch yaw">
     <xacro:include filename="$(find velodyne_description)/urdf/VLP-16.urdf.xacro"/>
-    <!-- <xacro:property name="pi" value="3.1415926835897931"/> -->
     <xacro:arg name="gpu" default="false"/>
     <xacro:property name="sensor_kit_base_link" default="sensor_kit_base_link"/>
