Commit message: chore: fix pre-commit
Signed-off-by: taikitanaka3 <taiki.tanaka@tier4.jp>

File: pandar_description/urdf/pandar_xt32.xacro (robot description, xacro)
@@ -31,6 +31,5 @@
         </geometry>
         <origin xyz="0 0 0.071" rpy="0 0 0"/>
-        <material name="gray">
-        </material>
+        <material name="gray"/>
       </visual>
       <visual>
@@ -39,6 +38,5 @@
         </geometry>
         <origin xyz="0.0 0.040 0.008" rpy="1.57 0 0"/>
-        <material name="gray">
-        </material>
+        <material name="gray"/>
       </visual>
       <inertial>
@@ -49,6 +47,6 @@
     </link>
     <joint name="${name}_base_scan_joint" type="fixed">
-      <origin xyz="0 0 0.0464" rpy="0 0 0" />
-      <parent link="${name}_base_link" />
+      <origin xyz="0 0 0.0464" rpy="0 0 0"/>
+      <parent link="${name}_base_link"/>
       <child link="${name}"/>
     </joint>
