Commit message: change visualization

File: pandar_description/urdf/pandar_ot128.xacro (robot description, xacro)
@@ -10,7 +10,7 @@
       <visual>
         <geometry>
-          <cylinder length="0.020" radius="0.040"/>
+          <cylinder length="0.05" radius="0.055"/>
         </geometry>
-        <origin xyz="0 0 0.010" rpy="0 0 0"/>
+        <origin xyz="0 0 0.025" rpy="0 0 0"/>
         <material name="gray">
           <color rgba="0.9 0.9 0.9 1.0"/>
@@ -19,23 +19,16 @@
       <visual>
         <geometry>
-          <cylinder length="0.046" radius="0.040"/>
+          <cylinder length="0.08" radius="0.053"/>
         </geometry>
-        <origin xyz="0 0 0.043" rpy="0 0 0"/>
-        <material name="blue">
-          <color rgba="0.0 0.0 1.0 1.0"/>
+        <origin xyz="0 0 0.09" rpy="0 0 0"/>
+        <material name="gray">
+          <color rgba="0.9 0.9 0.9 1.0"/>
         </material>
       </visual>
       <visual>
         <geometry>
-          <cylinder length="0.010" radius="0.040"/>
+          <cylinder length="0.006" radius="0.055"/>
         </geometry>
-        <origin xyz="0 0 0.071" rpy="0 0 0"/>
-        <material name="gray"/>
-      </visual>
-      <visual>
-        <geometry>
-          <cylinder length="0.030" radius="0.008"/>
-        </geometry>
-        <origin xyz="0.0 0.040 0.008" rpy="1.57 0 0"/>
+        <origin xyz="0 0 0.133" rpy="0 0 0"/>
         <material name="gray"/>
       </visual>
