Commit message: fix xacro & calibration

File: aip_x2_description/urdf/front_unit.xacro (robot description, xacro)
@@ -4,7 +4,6 @@
     <xacro:include filename="$(find pandar_description)/urdf/pandar_40p.xacro"/>
     <xacro:include filename="$(find pandar_description)/urdf/pandar_qt.xacro"/>
-    <!-- <xacro:property name="pi" value="3.1415926835897931"/> -->
     <xacro:arg name="gpu" default="false"/>
-    <xacro:arg name="config_dir" default="$(find aip_x2_description)"/>
+    <xacro:arg name="config_dir" default="$(find aip_x2_description)/config"/>
     <xacro:property name="front_unit_base_link" default="front_unit_base_link"/>
     <joint name="${front_unit_base_link}_joint" type="fixed">

File: aip_x2_description/urdf/rear_unit.xacro (robot description, xacro)
@@ -5,7 +5,6 @@
     <xacro:include filename="$(find pandar_description)/urdf/pandar_qt.xacro"/>
     <xacro:include filename="$(find camera_description)/urdf/monocular_camera.xacro"/>
-    <!-- <xacro:property name="pi" value="3.1415926835897931"/> -->
-    <xacro:arg name="gpu" default="false"/>
-    <xacro:arg name="config_dir" default="$(find aip_x2_description)"/>
+     <xacro:arg name="gpu" default="false"/>
+    <xacro:arg name="config_dir" default="$(find aip_x2_description)/config"/>
     <xacro:property name="rear_unit_base_link" default="rear_unit_base_link"/>
     <joint name="${rear_unit_base_link}_joint" type="fixed">

File: aip_x2_description/urdf/sensors.xacro (robot description, xacro)
@@ -2,13 +2,13 @@
 <robot name="vehicle"
   xmlns:xacro="http://ros.org/wiki/xacro">
-  <xacro:arg name="config_dir" default="$(find aip_x2_description)"/>
+  <xacro:arg name="config_dir" default="$(find aip_x2_description)/config"/>
   <xacro:property name="calibration" value="${load_yaml('$(arg config_dir)/sensors_calibration.yaml')}"/>
-  <!-- sensor kit -->
-  <xacro:include filename="sensor_kit.xacro"/>
-  <xacro:sensor_kit_macro parent="base_link" x="${calibration['base_link2sensor_kit_base_link']['x']}" y="${calibration['base_link2sensor_kit_base_link']['y']}" z="${calibration['base_link2sensor_kit_base_link']['z']}" roll="${calibration['base_link2sensor_kit_base_link']['roll']}" pitch="${calibration['base_link2sensor_kit_base_link']['pitch']}" yaw="${calibration['base_link2sensor_kit_base_link']['yaw']}" />
+  <!-- top unit -->
+  <xacro:include filename="top_unit.xacro"/>
+  <xacro:top_unit_macro parent="base_link" x="${calibration['base_link2top_unit_base_link']['x']}" y="${calibration['base_link2top_unit_base_link']['y']}" z="${calibration['base_link2top_unit_base_link']['z']}" roll="${calibration['base_link2top_unit_base_link']['roll']}" pitch="${calibration['base_link2top_unit_base_link']['pitch']}" yaw="${calibration['base_link2top_unit_base_link']['yaw']}" />
   <!-- front unit -->
   <xacro:include filename="front_unit.xacro"/>
   <xacro:front_unit_macro parent="base_link" x="${calibration['base_link2front_unit_base_link']['x']}" y="${calibration['base_link2front_unit_base_link']['y']}" z="${calibration['base_link2front_unit_base_link']['z']}" roll="${calibration['base_link2front_unit_base_link']['roll']}" pitch="${calibration['base_link2front_unit_base_link']['pitch']}" yaw="${calibration['base_link2front_unit_base_link']['yaw']}" />
-  <!-- rear -->
+  <!-- rear unit -->
   <xacro:include filename="rear_unit.xacro"/>
   <xacro:rear_unit_macro parent="base_link" x="${calibration['base_link2rear_unit_base_link']['x']}" y="${calibration['base_link2rear_unit_base_link']['y']}" z="${calibration['base_link2rear_unit_base_link']['z']}" roll="${calibration['base_link2rear_unit_base_link']['roll']}" pitch="${calibration['base_link2rear_unit_base_link']['pitch']}" yaw="${calibration['base_link2rear_unit_base_link']['yaw']}" />
