Commit message: fix suffix to name

File: camera_description/urdf/monocular_camera.xacro (robot description, xacro)
@@ -1,13 +1,13 @@
 <?xml version="1.0"?>
 <robot xmlns:xacro="http://ros.org/wiki/xacro">
-  <xacro:macro name="monocular_camera_macro" params="suffix parent namespace x y z roll pitch yaw fps width height fov">
+  <xacro:macro name="monocular_camera_macro" params="name parent namespace x y z roll pitch yaw fps width height fov">
     <xacro:property name="sensor_box" value="0.05" />
     <xacro:property name="mass" value="0.1" />
-    <joint name="${suffix}_joint" type="fixed">
+    <joint name="${name}_joint" type="fixed">
       <origin rpy="${roll} ${pitch} ${yaw}" xyz="${x} ${y} ${z}"/>
       <parent link="${parent}"/>
-      <child  link="${suffix}_link"/>
+      <child  link="${name}_link"/>
     </joint>
-    <link name="${suffix}_link">
+    <link name="${name}_link">
       <visual>
         <geometry>
@@ -33,16 +33,16 @@
       </collision>
     </link>
-    <joint name="${suffix}_optical_joint" type="fixed">
+    <joint name="${name}_optical_joint" type="fixed">
       <origin rpy="${-pi/2} 0 ${-pi/2}" xyz="0 0 0"/>
-      <parent link="${suffix}_link"/>
-      <child  link="${suffix}_optical_link"/>
+      <parent link="${name}_link"/>
+      <child  link="${name}_optical_link"/>
     </joint>
-    <link name="${suffix}_optical_link" />
+    <link name="${name}_optical_link" />
     <!-- camera -->
-    <gazebo reference="${suffix}_link">
+    <gazebo reference="${name}_link">
       <material>Gazebo/Black</material>
-      <sensor type="camera" name="${suffix}">
+      <sensor type="camera" name="${name}">
         <update_rate>${fps}</update_rate>
-        <camera name="${suffix}">
+        <camera name="${name}">
           <horizontal_fov>${fov}</horizontal_fov>
           <image>
@@ -70,5 +70,5 @@
           <imageTopicName>image_raw</imageTopicName>
           <cameraInfoTopicName>camera_info</cameraInfoTopicName>
-          <frameName>${suffix}_optical_link</frameName>
+          <frameName>${name}_optical_link</frameName>
           <hackBaseline>0.0</hackBaseline>
           <distortionK1>0.0</distortionK1>

File: imu_description/urdf/imu.xacro (robot description, xacro)
@@ -1,13 +1,13 @@
 <?xml version="1.0"?>
 <robot xmlns:xacro="http://ros.org/wiki/xacro">
-  <xacro:macro name="imu_macro" params="suffix parent namespace x y z roll pitch yaw fps">
+  <xacro:macro name="imu_macro" params="name parent namespace x y z roll pitch yaw fps">
     <xacro:property name="sensor_box" value="0.01" />
     <xacro:property name="mass" value="0.01" />
-    <joint name="${suffix}_joint" type="fixed">
+    <joint name="${name}_joint" type="fixed">
       <origin rpy="${roll} ${pitch} ${yaw}" xyz="${x} ${y} ${z}"/>
       <parent link="${parent}"/>
-      <child  link="${suffix}_link"/>
+      <child  link="${name}_link"/>
     </joint>
-    <link name="${suffix}_link">
+    <link name="${name}_link">
       <visual>
         <geometry>
@@ -34,7 +34,7 @@
     </link>
     <!-- imu -->
-    <gazebo reference="${suffix}_link">
+    <gazebo reference="${name}_link">
       <gravity>true</gravity>
-      <sensor name="${suffix}_sensor" type="imu">
+      <sensor name="${name}_sensor" type="imu">
         <always_on>true</always_on>
         <update_rate>${fps}</update_rate>
@@ -42,6 +42,6 @@
         <topic>__default_topic__</topic>
         <plugin filename="libgazebo_ros_imu_sensor.so" name="imu_plugin">
-          <topicName>${suffix}</topicName>
-          <bodyName>${suffix}_link</bodyName>
+          <topicName>${name}</topicName>
+          <bodyName>${name}_link</bodyName>
           <updateRateHZ>10.0</updateRateHZ>
           <gaussianNoise>0.0</gaussianNoise>

File: livox_description/urdf/livox_horizon.xacro (robot description, xacro)
@@ -1,13 +1,13 @@
 <?xml version="1.0"?>
 <robot xmlns:xacro="http://ros.org/wiki/xacro">
-  <xacro:macro name="livox_horizon_macro" params="suffix parent x y z roll pitch yaw">
+  <xacro:macro name="livox_horizon_macro" params="name parent x y z roll pitch yaw">
     <xacro:property name="sensor_box" value="0.1" />
     <xacro:property name="mass" value="0.01" />
-    <joint name="${suffix}_base_mount_joint" type="fixed">
+    <joint name="${name}_base_mount_joint" type="fixed">
       <origin rpy="${roll} ${pitch} ${yaw}" xyz="${x} ${y} ${z}"/>
       <parent link="${parent}"/>
-      <child  link="${suffix}_base_link"/>
+      <child  link="${name}_base_link"/>
     </joint>
-    <link name="${suffix}_base_link">
+    <link name="${name}_base_link">
       <visual>
         <geometry>
@@ -33,10 +33,10 @@
       </collision> -->
     </link>
-    <joint name="${suffix}_base_scan_joint" type="fixed" >
+    <joint name="${name}_base_scan_joint" type="fixed" >
       <origin xyz="0 0 0.0377" rpy="0 0 0" />
-      <parent link="${suffix}_base_link" />
-      <child link="${suffix}"/>
+      <parent link="${name}_base_link" />
+      <child link="${name}"/>
     </joint>
-    <link name="${suffix}">
+    <link name="${name}">
       <inertial>
         <mass value="0.0"/>

File: pandar_description/urdf/pandar_40p.xacro (robot description, xacro)
@@ -1,11 +1,11 @@
 <?xml version="1.0"?>
 <robot xmlns:xacro="http://ros.org/wiki/xacro">
-  <xacro:macro name="Pandar40P" params="suffix parent x y z roll pitch yaw">
-    <joint name="${suffix}_base_mount_joint" type="fixed">
+  <xacro:macro name="Pandar40P" params="name parent x y z roll pitch yaw">
+    <joint name="${name}_base_mount_joint" type="fixed">
       <origin rpy="${roll} ${pitch} ${yaw}" xyz="${x} ${y} ${z}"/>
       <parent link="${parent}"/>
-      <child  link="${suffix}_base_link"/>
+      <child  link="${name}_base_link"/>
     </joint>
-    <link name="${suffix}_base_link">
+    <link name="${name}_base_link">
       <visual>
         <geometry>
@@ -48,10 +48,10 @@
       </inertial>
     </link>
-    <joint name="${suffix}_base_scan_joint" type="fixed" >
+    <joint name="${name}_base_scan_joint" type="fixed" >
       <origin xyz="0 0 0.047" rpy="0 0 0" />
-      <parent link="${suffix}_base_link" />
-      <child link="${suffix}"/>
+      <parent link="${name}_base_link" />
+      <child link="${name}"/>
     </joint>
-    <link name="${suffix}">
+    <link name="${name}">
       <inertial>
         <mass value="0.0"/>

File: pandar_description/urdf/pandar_qt.xacro (robot description, xacro)
@@ -1,11 +1,11 @@
 <?xml version="1.0"?>
 <robot xmlns:xacro="http://ros.org/wiki/xacro">
-  <xacro:macro name="PandarQT" params="suffix parent x y z roll pitch yaw">
-    <joint name="${suffix}_base_mount_joint" type="fixed">
+  <xacro:macro name="PandarQT" params="name parent x y z roll pitch yaw">
+    <joint name="${name}_base_mount_joint" type="fixed">
       <origin rpy="${roll} ${pitch} ${yaw}" xyz="${x} ${y} ${z}"/>
       <parent link="${parent}"/>
-      <child  link="${suffix}_base_link"/>
+      <child  link="${name}_base_link"/>
     </joint>
-    <link name="${suffix}_base_link">
+    <link name="${name}_base_link">
       <visual>
         <geometry>
@@ -48,10 +48,10 @@
       </inertial>
     </link>
-    <joint name="${suffix}_base_scan_joint" type="fixed" >
+    <joint name="${name}_base_scan_joint" type="fixed" >
       <origin xyz="0 0 0.0504" rpy="0 0 0" />
-      <parent link="${suffix}_base_link" />
-      <child link="${suffix}"/>
+      <parent link="${name}_base_link" />
+      <child link="${name}"/>
     </joint>
-    <link name="${suffix}">
+    <link name="${name}">
       <inertial>
         <mass value="0.0"/>
