Commit message: ci(pre-commit): autofix

File: camera_description/urdf/monocular_camera.xacro (robot description, xacro)
@@ -2,10 +2,10 @@
 <robot xmlns:xacro="http://ros.org/wiki/xacro">
   <xacro:macro name="monocular_camera_macro" params="name parent namespace x y z roll pitch yaw fps width height fov">
-    <xacro:property name="sensor_box" value="0.05" />
-    <xacro:property name="mass" value="0.1" />
+    <xacro:property name="sensor_box" value="0.05"/>
+    <xacro:property name="mass" value="0.1"/>
     <joint name="${name}_joint" type="fixed">
       <origin rpy="${roll} ${pitch} ${yaw}" xyz="${x} ${y} ${z}"/>
       <parent link="${parent}"/>
-      <child  link="${name}_link"/>
+      <child link="${name}_link"/>
     </joint>
     <link name="${name}_link">
@@ -22,7 +22,12 @@
         <origin rpy="0 0 0" xyz="0 0 0"/>
         <mass value="${mass}"/>
-        <inertia ixx="${(sensor_box*sensor_box+sensor_box*sensor_box)*mass/12.0}" ixy="0.0" ixz="0.0"
-                 iyy="${(sensor_box*sensor_box+sensor_box*sensor_box)*mass/12.0}" iyz="0.0"
-                 izz="${(sensor_box*sensor_box+sensor_box*sensor_box)*mass/12.0}"/>
+        <inertia
+          ixx="${(sensor_box*sensor_box+sensor_box*sensor_box)*mass/12.0}"
+          ixy="0.0"
+          ixz="0.0"
+          iyy="${(sensor_box*sensor_box+sensor_box*sensor_box)*mass/12.0}"
+          iyz="0.0"
+          izz="${(sensor_box*sensor_box+sensor_box*sensor_box)*mass/12.0}"
+        />
       </inertial>
       <collision>
@@ -36,7 +41,7 @@
       <origin rpy="${-pi/2} 0 ${-pi/2}" xyz="0 0 0"/>
       <parent link="${name}_link"/>
-      <child  link="${name}_optical_link"/>
+      <child link="${name}_optical_link"/>
     </joint>
-    <link name="${name}_optical_link" />
+    <link name="${name}_optical_link"/>
     <!-- camera -->
     <gazebo reference="${name}_link">

File: imu_description/urdf/imu.xacro (robot description, xacro)
@@ -2,10 +2,10 @@
 <robot xmlns:xacro="http://ros.org/wiki/xacro">
   <xacro:macro name="imu_macro" params="name parent namespace x y z roll pitch yaw fps">
-    <xacro:property name="sensor_box" value="0.01" />
-    <xacro:property name="mass" value="0.01" />
+    <xacro:property name="sensor_box" value="0.01"/>
+    <xacro:property name="mass" value="0.01"/>
     <joint name="${name}_joint" type="fixed">
       <origin rpy="${roll} ${pitch} ${yaw}" xyz="${x} ${y} ${z}"/>
       <parent link="${parent}"/>
-      <child  link="${name}_link"/>
+      <child link="${name}_link"/>
     </joint>
     <link name="${name}_link">
@@ -22,7 +22,12 @@
         <origin rpy="0 0 0" xyz="0 0 0"/>
         <mass value="${mass}"/>
-        <inertia ixx="${(sensor_box*sensor_box+sensor_box*sensor_box)*mass/12.0}" ixy="0.0" ixz="0.0"
-                 iyy="${(sensor_box*sensor_box+sensor_box*sensor_box)*mass/12.0}" iyz="0.0"
-                 izz="${(sensor_box*sensor_box+sensor_box*sensor_box)*mass/12.0}"/>
+        <inertia
+          ixx="${(sensor_box*sensor_box+sensor_box*sensor_box)*mass/12.0}"
+          ixy="0.0"
+          ixz="0.0"
+          iyy="${(sensor_box*sensor_box+sensor_box*sensor_box)*mass/12.0}"
+          iyz="0.0"
+          izz="${(sensor_box*sensor_box+sensor_box*sensor_box)*mass/12.0}"
+        />
       </inertial>
       <!-- <collision>

File: livox_description/urdf/livox_horizon.xacro (robot description, xacro)
@@ -2,10 +2,10 @@
 <robot xmlns:xacro="http://ros.org/wiki/xacro">
   <xacro:macro name="livox_horizon_macro" params="name parent x y z roll pitch yaw">
-    <xacro:property name="sensor_box" value="0.1" />
-    <xacro:property name="mass" value="0.01" />
+    <xacro:property name="sensor_box" value="0.1"/>
+    <xacro:property name="mass" value="0.01"/>
     <joint name="${name}_base_mount_joint" type="fixed">
       <origin rpy="${roll} ${pitch} ${yaw}" xyz="${x} ${y} ${z}"/>
       <parent link="${parent}"/>
-      <child  link="${name}_base_link"/>
+      <child link="${name}_base_link"/>
     </joint>
     <link name="${name}_base_link">
@@ -22,7 +22,12 @@
         <origin rpy="0 0 0" xyz="0 0 0"/>
         <mass value="${mass}"/>
-        <inertia ixx="${(sensor_box*sensor_box+sensor_box*sensor_box)*mass/12.0}" ixy="0.0" ixz="0.0"
-                 iyy="${(sensor_box*sensor_box+sensor_box*sensor_box)*mass/12.0}" iyz="0.0"
-                 izz="${(sensor_box*sensor_box+sensor_box*sensor_box)*mass/12.0}"/>
+        <inertia
+          ixx="${(sensor_box*sensor_box+sensor_box*sensor_box)*mass/12.0}"
+          ixy="0.0"
+          ixz="0.0"
+          iyy="${(sensor_box*sensor_box+sensor_box*sensor_box)*mass/12.0}"
+          iyz="0.0"
+          izz="${(sensor_box*sensor_box+sensor_box*sensor_box)*mass/12.0}"
+        />
       </inertial>
       <!-- <collision>
@@ -33,7 +38,7 @@
       </collision> -->
     </link>
-    <joint name="${name}_base_scan_joint" type="fixed" >
-      <origin xyz="0 0 0.0377" rpy="0 0 0" />
-      <parent link="${name}_base_link" />
+    <joint name="${name}_base_scan_joint" type="fixed">
+      <origin xyz="0 0 0.0377" rpy="0 0 0"/>
+      <parent link="${name}_base_link"/>
       <child link="${name}"/>
     </joint>

File: pandar_description/urdf/pandar_40p.xacro (robot description, xacro)
@@ -5,5 +5,5 @@
       <origin rpy="${roll} ${pitch} ${yaw}" xyz="${x} ${y} ${z}"/>
       <parent link="${parent}"/>
-      <child  link="${name}_base_link"/>
+      <child link="${name}_base_link"/>
     </joint>
     <link name="${name}_base_link">
@@ -31,6 +31,5 @@
         </geometry>
         <origin xyz="0 0 0.094" rpy="0 0 0"/>
-        <material name="gray">
-        </material>
+        <material name="gray"/>
       </visual>
       <visual>
@@ -39,6 +38,5 @@
         </geometry>
         <origin xyz="0.0 0.059 0.010" rpy="1.57 0 0"/>
-        <material name="gray">
-        </material>
+        <material name="gray"/>
       </visual>
       <inertial>
@@ -48,7 +46,7 @@
       </inertial>
     </link>
-    <joint name="${name}_base_scan_joint" type="fixed" >
-      <origin xyz="0 0 0.047" rpy="0 0 0" />
-      <parent link="${name}_base_link" />
+    <joint name="${name}_base_scan_joint" type="fixed">
+      <origin xyz="0 0 0.047" rpy="0 0 0"/>
+      <parent link="${name}_base_link"/>
       <child link="${name}"/>
     </joint>

File: pandar_description/urdf/pandar_qt.xacro (robot description, xacro)
@@ -5,5 +5,5 @@
       <origin rpy="${roll} ${pitch} ${yaw}" xyz="${x} ${y} ${z}"/>
       <parent link="${parent}"/>
-      <child  link="${name}_base_link"/>
+      <child link="${name}_base_link"/>
     </joint>
     <link name="${name}_base_link">
@@ -31,6 +31,5 @@
         </geometry>
         <origin xyz="0 0 0.071" rpy="0 0 0"/>
-        <material name="gray">
-        </material>
+        <material name="gray"/>
       </visual>
       <visual>
@@ -39,6 +38,5 @@
         </geometry>
         <origin xyz="0.0 0.040 0.008" rpy="1.57 0 0"/>
-        <material name="gray">
-        </material>
+        <material name="gray"/>
       </visual>
       <inertial>
@@ -48,7 +46,7 @@
       </inertial>
     </link>
-    <joint name="${name}_base_scan_joint" type="fixed" >
-      <origin xyz="0 0 0.0504" rpy="0 0 0" />
-      <parent link="${name}_base_link" />
+    <joint name="${name}_base_scan_joint" type="fixed">
+      <origin xyz="0 0 0.0504" rpy="0 0 0"/>
+      <parent link="${name}_base_link"/>
       <child link="${name}"/>
     </joint>

File: velodyne_description/urdf/HDL-32E.urdf.xacro (robot description, xacro)
@@ -1,8 +1,11 @@
 <?xml version="1.0"?>
 <robot xmlns:xacro="http://www.ros.org/wiki/xacro" name="HDL-32E">
-  <xacro:property name="M_PI" value="3.1415926535897931" />
-  <xacro:macro name="HDL-32E" params="*origin parent:=base_link name:=velodyne tf_prefix:='' topic:=/velodyne_points organize_cloud:=false hz:=10 lasers:=32 samples:=2187 collision_range:=0.3 min_range:=0.9 max_range:=130.0 noise:=0.008 min_angle:=-${M_PI} max_angle:=${M_PI} gpu:=false">
+  <xacro:property name="M_PI" value="3.1415926535897931"/>
+  <xacro:macro
+    name="HDL-32E"
+    params="*origin parent:=base_link name:=velodyne tf_prefix:='' topic:=/velodyne_points organize_cloud:=false hz:=10 lasers:=32 samples:=2187 collision_range:=0.3 min_range:=0.9 max_range:=130.0 noise:=0.008 min_angle:=-${M_PI} max_angle:=${M_PI} gpu:=false"
+  >
     <joint name="${name}_base_mount_joint" type="fixed">
-      <xacro:insert_block name="origin" />
+      <xacro:insert_block name="origin"/>
       <parent link="${parent}"/>
       <child link="${name}_base_link"/>
@@ -12,11 +15,16 @@
         <mass value="1.0"/>
         <origin xyz="0 0 0.07212"/>
-        <inertia ixx="${(1.0 * (3.0*0.04267*0.04267 + 0.14424*0.14424)) / 12.0}" ixy="0" ixz="0"
-          iyy="${(1.0 * (3.0*0.04267*0.04267 + 0.14424*0.14424)) / 12.0}" iyz="0"
-          izz="${0.5 * 1.0 * (0.04267*0.04267)}"/>
+        <inertia
+          ixx="${(1.0 * (3.0*0.04267*0.04267 + 0.14424*0.14424)) / 12.0}"
+          ixy="0"
+          ixz="0"
+          iyy="${(1.0 * (3.0*0.04267*0.04267 + 0.14424*0.14424)) / 12.0}"
+          iyz="0"
+          izz="${0.5 * 1.0 * (0.04267*0.04267)}"
+        />
       </inertial>
       <visual>
         <geometry>
-          <mesh filename="package://velodyne_description/meshes/HDL32E_base.dae" />
+          <mesh filename="package://velodyne_description/meshes/HDL32E_base.dae"/>
         </geometry>
       </visual>
@@ -28,7 +36,7 @@
       </collision>
     </link>
-    <joint name="${name}_base_scan_joint" type="fixed" >
-      <origin xyz="0 0 0.09081" rpy="0 0 0" />
-      <parent link="${name}_base_link" />
+    <joint name="${name}_base_scan_joint" type="fixed">
+      <origin xyz="0 0 0.09081" rpy="0 0 0"/>
+      <parent link="${name}_base_link"/>
       <child link="${name}"/>
     </joint>
@@ -40,7 +48,7 @@
       </inertial>
       <visual>
-        <origin xyz="0 0 -0.09081" rpy="0 0 0" />
+        <origin xyz="0 0 -0.09081" rpy="0 0 0"/>
         <geometry>
-          <mesh filename="package://velodyne_description/meshes/HDL32E_scan.dae" />
+          <mesh filename="package://velodyne_description/meshes/HDL32E_scan.dae"/>
         </geometry>
       </visual>
@@ -65,5 +73,5 @@
                 <resolution>1</resolution>
                 <min_angle>-${30.67*M_PI/180.0}</min_angle>
-                <max_angle> ${10.67*M_PI/180.0}</max_angle>
+                <max_angle>${10.67*M_PI/180.0}</max_angle>
               </vertical>
             </scan>
@@ -110,5 +118,5 @@
                 <resolution>1</resolution>
                 <min_angle>-${30.67*M_PI/180.0}</min_angle>
-                <max_angle> ${10.67*M_PI/180.0}</max_angle>
+                <max_angle>${10.67*M_PI/180.0}</max_angle>
               </vertical>
             </scan>

File: velodyne_description/urdf/VLP-16.urdf.xacro (robot description, xacro)
@@ -1,8 +1,11 @@
 <?xml version="1.0"?>
 <robot xmlns:xacro="http://www.ros.org/wiki/xacro" name="VLP-16">
-  <xacro:property name="M_PI" value="3.1415926535897931" />
-  <xacro:macro name="VLP-16" params="*origin parent:=base_link name:=velodyne tf_prefix:='' topic:=/velodyne_points organize_cloud:=false hz:=10 lasers:=16 samples:=1875 collision_range:=0.3 min_range:=0.9 max_range:=130.0 noise:=0.008 min_angle:=-${M_PI} max_angle:=${M_PI} gpu:=false">
+  <xacro:property name="M_PI" value="3.1415926535897931"/>
+  <xacro:macro
+    name="VLP-16"
+    params="*origin parent:=base_link name:=velodyne tf_prefix:='' topic:=/velodyne_points organize_cloud:=false hz:=10 lasers:=16 samples:=1875 collision_range:=0.3 min_range:=0.9 max_range:=130.0 noise:=0.008 min_angle:=-${M_PI} max_angle:=${M_PI} gpu:=false"
+  >
     <joint name="${name}_base_mount_joint" type="fixed">
-      <xacro:insert_block name="origin" />
+      <xacro:insert_block name="origin"/>
       <parent link="${parent}"/>
       <child link="${name}_base_link"/>
@@ -12,16 +15,21 @@
         <mass value="0.83"/>
         <origin xyz="0 0 0.03585"/>
-        <inertia ixx="${(0.83 * (3.0*0.0516*0.0516 + 0.0717*0.0717)) / 12.0}" ixy="0" ixz="0"
-          iyy="${(0.83 * (3.0*0.0516*0.0516 + 0.0717*0.0717)) / 12.0}" iyz="0"
-          izz="${0.5 * 0.83 * (0.0516*0.0516)}"/>
+        <inertia
+          ixx="${(0.83 * (3.0*0.0516*0.0516 + 0.0717*0.0717)) / 12.0}"
+          ixy="0"
+          ixz="0"
+          iyy="${(0.83 * (3.0*0.0516*0.0516 + 0.0717*0.0717)) / 12.0}"
+          iyz="0"
+          izz="${0.5 * 0.83 * (0.0516*0.0516)}"
+        />
       </inertial>
       <visual>
         <geometry>
-          <mesh filename="package://velodyne_description/meshes/VLP16_base_1.dae" />
+          <mesh filename="package://velodyne_description/meshes/VLP16_base_1.dae"/>
         </geometry>
       </visual>
       <visual>
         <geometry>
-          <mesh filename="package://velodyne_description/meshes/VLP16_base_2.dae" />
+          <mesh filename="package://velodyne_description/meshes/VLP16_base_2.dae"/>
         </geometry>
       </visual>
@@ -33,7 +41,7 @@
       </collision>
     </link>
-    <joint name="${name}_base_scan_joint" type="fixed" >
-      <origin xyz="0 0 0.0377" rpy="0 0 0" />
-      <parent link="${name}_base_link" />
+    <joint name="${name}_base_scan_joint" type="fixed">
+      <origin xyz="0 0 0.0377" rpy="0 0 0"/>
+      <parent link="${name}_base_link"/>
       <child link="${name}"/>
     </joint>
@@ -45,7 +53,7 @@
       </inertial>
       <visual>
-        <origin xyz="0 0 -0.0377" />
+        <origin xyz="0 0 -0.0377"/>
         <geometry>
-          <mesh filename="package://velodyne_description/meshes/VLP16_scan.dae" />
+          <mesh filename="package://velodyne_description/meshes/VLP16_scan.dae"/>
         </geometry>
       </visual>
@@ -70,5 +78,5 @@
                 <resolution>1</resolution>
                 <min_angle>-${15.0*M_PI/180.0}</min_angle>
-                <max_angle> ${15.0*M_PI/180.0}</max_angle>
+                <max_angle>${15.0*M_PI/180.0}</max_angle>
               </vertical>
             </scan>
@@ -115,5 +123,5 @@
                 <resolution>1</resolution>
                 <min_angle>-${15.0*M_PI/180.0}</min_angle>
-                <max_angle> ${15.0*M_PI/180.0}</max_angle>
+                <max_angle>${15.0*M_PI/180.0}</max_angle>
               </vertical>
             </scan>

File: velodyne_description/urdf/example.urdf.xacro (robot description, xacro)
@@ -2,24 +2,24 @@
 <robot xmlns:xacro="http://www.ros.org/wiki/xacro" name="example">
   <xacro:arg name="gpu" default="false"/>
-  <xacro:property name="gpu" value="$(arg gpu)" />
+  <xacro:property name="gpu" value="$(arg gpu)"/>
   <xacro:arg name="organize_cloud" default="false"/>
-  <xacro:property name="organize_cloud" value="$(arg organize_cloud)" />
+  <xacro:property name="organize_cloud" value="$(arg organize_cloud)"/>
   <!-- Base Footprint -->
-  <link name="base_footprint" />
+  <link name="base_footprint"/>
   <!-- Base Link -->
-  <joint name="footprint" type="fixed" >
-   <parent link="base_footprint" />
-    <child link="base_link" />
-    <origin xyz="0 0 0.05" rpy="0 0 0" />
+  <joint name="footprint" type="fixed">
+    <parent link="base_footprint"/>
+    <child link="base_link"/>
+    <origin xyz="0 0 0.05" rpy="0 0 0"/>
   </joint>
-  <link name="base_link" >
+  <link name="base_link">
     <visual>
       <geometry>
-        <box size="0.5 0.5 0.1" />
+        <box size="0.5 0.5 0.1"/>
       </geometry>
     </visual>
     <collision>
       <geometry>
-        <box size="0.5 0.5 0.1" />
+        <box size="0.5 0.5 0.1"/>
       </geometry>
     </collision>
@@ -27,16 +27,14 @@
       <origin xyz="0 0 0"/>
       <mass value="10"/>
-      <inertia ixx="3.0" ixy="0.0" ixz="0.0"
-               iyy="3.0" iyz="0.0"
-               izz="3.0" />
+      <inertia ixx="3.0" ixy="0.0" ixz="0.0" iyy="3.0" iyz="0.0" izz="3.0"/>
     </inertial>
   </link>
   <xacro:include filename="$(find velodyne_description)/urdf/VLP-16.urdf.xacro"/>
   <xacro:VLP-16 parent="base_link" name="velodyne" topic="/velodyne_points" organize_cloud="${organize_cloud}" hz="10" samples="440" gpu="${gpu}">
-    <origin xyz="0 0 0.4" rpy="0 0 0" />
+    <origin xyz="0 0 0.4" rpy="0 0 0"/>
   </xacro:VLP-16>
   <xacro:include filename="$(find velodyne_description)/urdf/HDL-32E.urdf.xacro"/>
   <xacro:HDL-32E parent="base_link" name="velodyne2" topic="/velodyne_points2" organize_cloud="${organize_cloud}" hz="10" samples="220" gpu="${gpu}">
-    <origin xyz="0 0 0.6" rpy="0 0 0" />
+    <origin xyz="0 0 0.6" rpy="0 0 0"/>
   </xacro:HDL-32E>
 </robot>

File: vls_description/urdf/VLS-128.urdf.xacro (robot description, xacro)
@@ -2,5 +2,8 @@
 <robot xmlns:xacro="http://www.ros.org/wiki/xacro" name="VLS-128">
   <xacro:property name="M_PI" value="3.1415926535897931"/>
-  <xacro:macro name="VLS-128" params="*origin parent:=base_link name:=velodyne topic:=/velodyne_points hz:=10 lasers:=128 samples:=1875 collision_range:=0.3 min_range:=0.9 max_range:=130.0 noise:=0.008 min_angle:=-${M_PI} max_angle:=${M_PI} gpu:=false">
+  <xacro:macro
+    name="VLS-128"
+    params="*origin parent:=base_link name:=velodyne topic:=/velodyne_points hz:=10 lasers:=128 samples:=1875 collision_range:=0.3 min_range:=0.9 max_range:=130.0 noise:=0.008 min_angle:=-${M_PI} max_angle:=${M_PI} gpu:=false"
+  >
     <joint name="${name}_base_mount_joint" type="fixed">
       <xacro:insert_block name="origin"/>
@@ -12,5 +15,12 @@
         <mass value="3.53"/>
         <origin xyz="0 0 0.07065"/>
-        <inertia ixx="${(3.53 * (3.0*0.0827*0.0827 + 0.1413*0.1413)) / 12.0}" ixy="0" ixz="0" iyy="${(3.53 * (3.0*0.0827*0.0827 + 0.1413*0.1413)) / 12.0}" iyz="0" izz="${0.5 * 3.53 * (0.0827*0.0827)}"/>
+        <inertia
+          ixx="${(3.53 * (3.0*0.0827*0.0827 + 0.1413*0.1413)) / 12.0}"
+          ixy="0"
+          ixz="0"
+          iyy="${(3.53 * (3.0*0.0827*0.0827 + 0.1413*0.1413)) / 12.0}"
+          iyz="0"
+          izz="${0.5 * 3.53 * (0.0827*0.0827)}"
+        />
       </inertial>
       <visual>
@@ -68,6 +78,5 @@
                 <resolution>1</resolution>
                 <min_angle>-${25.0*M_PI/180.0}</min_angle>
-                <max_angle>
-                  ${15.0*M_PI/180.0}</max_angle>
+                <max_angle>${15.0*M_PI/180.0}</max_angle>
               </vertical>
             </scan>
@@ -109,6 +118,5 @@
                 <resolution>1</resolution>
                 <min_angle>-${25.0*M_PI/180.0}</min_angle>
-                <max_angle>
-                  ${15.0*M_PI/180.0}</max_angle>
+                <max_angle>${15.0*M_PI/180.0}</max_angle>
               </vertical>
             </scan>
