Commit message: Modify m1600ex optical center in x/y direction

File: velarray_description/urdf/velarray_m1600ex.xacro (robot description, xacro)
@@ -33,6 +33,6 @@
     </link>
     <joint name="${name}_base_scan_joint" type="fixed">
-      <!-- NOTE: optical center is actually difference from the base_link in x/y direction -->
-      <origin xyz="0 0 0.0275" rpy="0 0 0" />
+      <!-- NOTE: base_link is described as "DATUM A" in datasheet -->
+      <origin xyz="0.04972 -0.03619 0.0275" rpy="0 0 0" />
       <parent link="${name}_base_link" />
       <child link="${name}"/>

Commit message: Modify m1600ex base_link definition
Signed-off-by: Akihito OHSATO <aohsato@gmail.com>

File: velarray_description/urdf/velarray_m1600ex.xacro (robot description, xacro)
@@ -32,6 +32,7 @@
       </collision> -->
     </link>
+    <!-- base_link is the bottom of the optical center -->
     <joint name="${name}_base_scan_joint" type="fixed">
-      <origin xyz="0.04972 -0.03619 0.0275" rpy="0 0 0" />
+      <origin xyz="0.0 0.0 0.0275" rpy="0 0 0" />
       <parent link="${name}_base_link" />
       <child link="${name}"/>
