Commit message: ci(pre-commit): autofix

File: radar_description/urdf/radar.xacro (robot description, xacro)
@@ -2,9 +2,9 @@
 <robot xmlns:xacro="http://ros.org/wiki/xacro">
   <xacro:macro name="radar_macro" params="name parent x y z roll pitch yaw">
-    <xacro:property name="mass" value="0.01" />
+    <xacro:property name="mass" value="0.01"/>
     <joint name="${name}_base_mount_joint" type="fixed">
       <origin rpy="${roll} ${pitch} ${yaw}" xyz="${x} ${y} ${z}"/>
       <parent link="${parent}"/>
-      <child  link="${name}_base_link"/>
+      <child link="${name}_base_link"/>
     </joint>
     <link name="${name}_base_link">
@@ -21,7 +21,5 @@
         <origin rpy="0 0 0" xyz="0 0 0"/>
         <mass value="${mass}"/>
-        <inertia ixx="${(0.03*0.03+0.03*0.03)*mass/12.0}" ixy="0.0" ixz="0.0"
-                 iyy="${(0.1*0.1+0.1*0.1)*mass/12.0}" iyz="0.0"
-                 izz="${(0.1*0.1+0.1*0.1)*mass/12.0}"/>
+        <inertia ixx="${(0.03*0.03+0.03*0.03)*mass/12.0}" ixy="0.0" ixz="0.0" iyy="${(0.1*0.1+0.1*0.1)*mass/12.0}" iyz="0.0" izz="${(0.1*0.1+0.1*0.1)*mass/12.0}"/>
       </inertial>
     </link>

Commit message: fix: fixed the radar names. there is no base link in the radars
Signed-off-by: Kenzo Lobos-Tsunekawa <kenzo.lobos@tier4.jp>

File: radar_description/urdf/radar.xacro (robot description, xacro)
@@ -6,7 +6,7 @@
       <origin rpy="${roll} ${pitch} ${yaw}" xyz="${x} ${y} ${z}"/>
       <parent link="${parent}"/>
-      <child link="${name}_base_link"/>
+      <child link="${name}"/>
     </joint>
-    <link name="${name}_base_link">
+    <link name="${name}">
       <visual>
         <geometry>
